Commit message: assignment 3 complete

File: urdf/athens.urdf (robot description, URDF)
Before this commit: robot athens, 1 links, 0 joints
Links:
- added link arm_0_link; collision cylinder length=0.4 radius=0.05; visual cylinder length=0.4 radius=0.05
- added link arm_1_link; collision cylinder length=0.4 radius=0.05; visual cylinder length=0.4 radius=0.05
- added link arm_2_link; collision cylinder length=0.4 radius=0.05; visual cylinder length=0.4 radius=0.05
- added link gripper_1_link; collision box size=0.02 0.05 0.1; visual box size=0.02 0.05 0.1
- added link gripper_2_link; collision box size=0.02 0.05 0.1; visual box size=0.02 0.05 0.1
- added link gripper_base_link; collision box size=0.1 0.1 0.05; visual box size=0.1 0.1 0.05
- link base_link: geometry collision cylinder length=0.5 radius=0.1; visual cylinder length=0.5 radius=0.1
Joints:
- added joint arm_0_joint: type revolute, parent base_link, child arm_0_link, origin xyz=0 0 0.5 rpy=0 0 0, axis 0 1 0, limit lower=-1.57 upper=1.57 effort=10 velocity=1
- added joint arm_1_joint: type revolute, parent arm_0_link, child arm_1_link, origin xyz=0 0 0.4 rpy=0 0 0, axis 0 1 0, limit lower=-1.57 upper=1.57 effort=10 velocity=1
- added joint arm_2_joint: type revolute, parent arm_1_link, child arm_2_link, origin xyz=0 0 0.4 rpy=0 0 0, axis 0 1 0, limit lower=-1.57 upper=1.57 effort=10 velocity=1
- added joint gripper_1_joint: type prismatic, parent gripper_base_link, child gripper_1_link, origin xyz=0.04 0 0.07 rpy=0 0 0, axis 1 0 0, limit lower=0 upper=0.05 effort=10 velocity=0.1
- added joint gripper_2_joint: type prismatic, parent gripper_base_link, child gripper_2_link, origin xyz=-0.04 0 0.07 rpy=0 0 0, axis -1 0 0, limit lower=0 upper=0.05 effort=10 velocity=0.1
- added joint gripper_base_joint: type fixed, parent arm_2_link, child gripper_base_link, origin xyz=0 0 0.425 rpy=0 0 0
